Commit message: good dometry and control in simulator

File: homere_description/urdf/homere.urdf (robot description, URDF)
Before this commit: robot homere, 2 links, 1 joints
Links:
- link imu_link: geometry visual box size=0.1 0.1 0.1

File: homere_simulator/urdf/homere.urdf.xacro (robot description, xacro)
@@ -19,9 +19,32 @@
       <robotParam>robot_description</robotParam>
       <controlPeriod>0.01</controlPeriod>
-      <robotSimType>gazebo_ros_control/DefaultRobotHWSim</robotSimType>
+      <!--<robotSimType>gazebo_ros_control/DefaultRobotHWSim</robotSimType>-->
+      <robotSimType>homere_simulator/HomereHardwareInterface</robotSimType>
     </plugin>
   </gazebo>
+  <gazebo>
+    <plugin name="ground_truth" filename="libgazebo_ros_p3d.so">
+      <frameName>world</frameName>
+      <bodyName>base_link</bodyName>
+      <topicName>homere/base_link_truth</topicName>
+      <updateRate>30.0</updateRate>
+    </plugin>
+  </gazebo>
+  <!-- GazeboRosImu -->
   <!--
-  <gazebo reference="imu_link">
+  <gazebo>
+    <plugin name="imu_plugin" filename="libgazebo_ros_imu.so">
+      <robotNamespace>homere</robotNamespace>
+      <alwaysOn>true</alwaysOn>
+      <bodyName>imu_link</bodyName>
+      <topicName>imu</topicName>
+      <serviceName>imu_service</serviceName>
+      <gaussianNoise>0.0</gaussianNoise>
+      <updateRate>100.0</updateRate>
+    </plugin>
+  </gazebo>
+  -->
+  <!-- GazeboRosImuSensor -->
+    <gazebo reference="imu_link">
     <gravity>true</gravity>
     <sensor name="imu_sensor" type="imu">
@@ -31,7 +54,8 @@
       <topic>__default_topic__</topic>
       <plugin filename="libgazebo_ros_imu_sensor.so" name="imu_plugin">
-        <topicName>imu</topicName>
+        <robotNamespace>/homere</robotNamespace>
+	<topicName>imu</topicName>
         <bodyName>imu_link</bodyName>
-        <updateRateHZ>10.0</updateRateHZ>
+        <updateRateHZ>100.0</updateRateHZ>
         <gaussianNoise>0.0</gaussianNoise>
         <xyzOffset>0 0 0</xyzOffset>
@@ -41,7 +65,28 @@
       <pose>0 0 0 0 0 0</pose>
     </sensor>
-    </gazebo>
+  </gazebo>
+  <!--
+  <gazebo>
+    <plugin name="imu_plugin" filename="libgazebo_ros_imu.so">
+      <always_on>true</always_on>
+      <updateRate>100.0</updateRate>
+      <bodyName>imu_link</bodyName>
+      <topicName>imu</topicName>
+      <gaussianNoise>0.0</gaussianNoise>
+      <xyzOffset>0 0 0</xyzOffset>
+      <rpyOffset>0 0 0</rpyOffset>
+      <serviceName>imu_service</serviceName>
+    </plugin>
+  </gazebo>
+  <gazebo reference="imu_link">
+    <sensor name="imu_sensor" type="imu">
+      <always_on>true</always_on>
+      <update_rate>100</update_rate>
+      <visualize>true</visualize>
+      <topic>__default_topic__</topic>
+    </sensor>
+  </gazebo>
   -->
-  <!-- -->
+  <!--
  <gazebo reference="imu_link">
  </gazebo>
@@ -57,5 +102,5 @@
     </plugin>
   </gazebo>
-  <!-- -->
+  -->
   <!--
     <gazebo reference="imu_link">

Commit message: lots... odometry, control

File: homere_description/urdf/homere.urdf (robot description, URDF)
Before this commit: robot homere, 2 links, 1 joints
Links:
- link imu_link: geometry visual sphere radius=0.025
